Commit message: Update spawn launch files, remove test models, add new models and worlds

File: src/tortoise_bot/urdf/turtlebot3_burger_cam.urdf (robot description, URDF)
Before this commit: robot turtlebot3_burger_cam, 10 links, 9 joints
Links:
- link base_link: geometry collision box size=0.140 0.140 0.143; visual mesh filename=package://tortoise_bot/models/turtlebot3_common/meshes/base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 scale=0.001 0.001 0.001
- link base_scan: geometry collision cylinder length=0.0315 radius=0.055; visual mesh filename=package://tortoise_bot/models/turtlebot3_common/meshes/sens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 scale=0.001 0.001 0.001
- link wheel_left_link: geometry collision cylinder length=0.018 radius=0.033; visual mesh filename=package://tortoise_bot/models/turtlebot3_common/meshes/whee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 scale=0.001 0.001 0.001
- link wheel_right_link: geometry collision cylinder length=0.018 radius=0.033; visual mesh filename=package://tortoise_bot/models/turtlebot3_common/meshes/whee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 scale=0.001 0.001 0.001
